Commit message: 第6章完成

File: ws_zxz_chapt6/src/cpp01_urdf/urdf/xacro/xacro_car/car_base.xacro (robot description, xacro)
@@ -10,4 +10,6 @@
   <!-- 离地间距 0.025+0.035=0.06 -->
   <xacro:property name="distance" value="${wheel_radius + car_height / 2}"/>
+  <!-- 车轮偏移 -->
+  <xacro:property name="wheel_offset" value="0.06"/>
   <!-- set color -->
   <material name="yellow">
@@ -16,4 +18,10 @@
   <material name="black">
     <color rgba="0.0 0.0 0.0 0.5"/>
+  </material>
+  <material name="red">
+    <color rgba="0.8 0.1 0.1 0.8"/>
+  </material>
+  <material name="pink">
+    <color rgba="0.4 0.2 0.6 0.8"/>
   </material>
   <!-- set base_footprint -->
@@ -40,6 +48,7 @@
     <origin xyz="0.0 0.0 ${distance}"/>
   </joint>
-  <!-- 定义车轮宏 -->
+  <!-- 定义车轮宏(创建车轮, 和车轮关节 -->
   <xacro:macro name="wheel_create" params="wheel_name is_front is_left">
+    <!-- 创建车轮 -->
     <link name="${wheel_name}">
       <visual>
@@ -48,5 +57,5 @@
           <cylinder radius="${wheel_radius}" length="${wheel_length}"/>
         </geometry>
-        <!-- 设置偏移 -->
+        <!-- 角度设置偏移 -->
         <origin rpy="${PI / 2} 0 0"/>
         <!-- 设置颜色 -->
@@ -54,7 +63,16 @@
       </visual>
     </link>
+    <!-- 配置关节 -->
+    <joint name="${wheel_name}_to_baselink" type="continuous">
+      <origin xyz="${wheel_offset * is_front} ${wheel_offset * is_left} -0.035"/>
+      <parent link="base_link"/>
+      <child link="${wheel_name}"/>
+      <axis xyz="0 1 0"/>
+    </joint>
   </xacro:macro>
-  <!-- 定义车轮与baselink连接宏 -->
-  <xacro:macro name="wheel_link" params="wheel_name wheel_origin">
-  </xacro:macro>
+  <!-- 车轮宏调用 -->
+  <xacro:wheel_create wheel_name="left_front_wheel" is_front="1" is_left="1"/>
+  <xacro:wheel_create wheel_name="right_front_wheel" is_front="1" is_left="-1"/>
+  <xacro:wheel_create wheel_name="left_back_wheel" is_front="-1" is_left="1"/>
+  <xacro:wheel_create wheel_name="right_back_wheel" is_front="-1" is_left="-1"/>
 </robot>

File: ws_zxz_chapt6/src/cpp01_urdf/urdf/xacro/xacro_car/car_camera.xacro (robot description, xacro)
@@ -1,3 +1,26 @@
 <!-- 摄像头 -->
 <robot xmlns:xacro="http://wiki.ros.org/xacro">
+  <!-- 声明变量 -->
+  <xacro:property name="camera_x" value="0.012"/>
+  <xacro:property name="camera_y" value="0.05"/>
+  <xacro:property name="camera_z" value="0.01"/>
+  <xacro:property name="camera_x_offset" value="${car_length / 2 - camera_x / 2}"/>
+  <xacro:property name="camera_y_offset" value="0.0"/>
+  <xacro:property name="camera_z_offset" value="${car_height / 2 + camera_z / 2}"/>
+  <!-- 创建照相机模型 -->
+  <link name="camera">
+    <visual>
+      <geometry>
+        <box size="${camera_x} ${camera_y} ${camera_z}"/>
+      </geometry>
+      <origin xyz="0.0 0.0 0.0" rpy="0.0 0.0 0.0" />
+      <material name="red"/>
+    </visual>
+  </link>
+  <!-- 创建照相机关节 -->
+  <joint name="camera_to_baselink" type="fixed">
+    <parent link="base_link"/>
+    <child link="camera"/>
+    <origin xyz="${camera_x_offset} ${camera_y_offset} ${camera_z_offset}" rpy="0.0 0.0 0.0"/>
+  </joint>
 </robot>

File: ws_zxz_chapt6/src/cpp01_urdf/urdf/xacro/xacro_car/car_laser.xacro (robot description, xacro)
@@ -1,3 +1,23 @@
 <!-- 雷达 -->
 <robot xmlns:xacro="http://wiki.ros.org/xacro">
+  <xacro:property name="laser_radius" value="0.03"/>
+  <xacro:property name="laser_length" value="0.03"/>
+  <xacro:property name="laser_x_offset" value="0.0"/>
+  <xacro:property name="laser_y_offset" value="0.0"/>
+  <xacro:property name="laser_z_offset" value="${car_height / 2 + laser_length / 2}"/>
+  <link name="laser">
+    <visual>
+      <geometry>
+        <cylinder radius="${laser_radius}" length="${laser_length}"/>
+      </geometry>
+      <material name="pink"/>
+      <origin xyz="0.0 0.0 0.0" rpy="0.0 0.0 0.0"/>
+    </visual>
+  </link>
+  <joint name="laser_to_baselink" type="continuous">
+    <parent link="base_link"/>
+    <child link="laser"/>
+    <axis xyz="0 0 1"/>
+    <origin xyz="${laser_x_offset} ${laser_y_offset} ${laser_z_offset}" rpy="0.0 0.0 0.0"/>
+  </joint>
 </robot>
